File: Parasite.brd (EAGLE design)
At the start: 61 x 64.1 mm, 63 parts, among them SW0 3_PIN_CONNECTOR, SW1 3_PIN_CONNECTOR, SW2 3_PIN_CONNECTOR, SW3 3_PIN_CONNECTOR, U1 ATMEGA328PB-AU, U2 DIGITAL_POT_AD5242AD5242/AD52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, U3 DIGITAL_POT_AD5282AD5242/AD52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, U4 DIGITAL_POT_AD5242AD5242/AD52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, U5 TMUX1134, U6 7_SEGMENT_DISPLAY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

Commit message: Finished v1 layout
Parts:
- moved C10 44.4 mm to (53.3, 42.5)
- moved U5 43.3 mm to (53.3, 35.1)
- moved SJ2 27.8 mm to (2.54, 29.7)
- moved SJ3 27.7 mm to (17.8, 30.0)
- moved SJ1 26.5 mm to (33.0, 29.8)
- moved R6 18.1 mm to (15.2, 47.0), flipped to the top
- moved R11 16.5 mm to (29.2, 40.0), turned to 270 degrees
- moved R4 16.5 mm to (36.8, 40.0), turned to 270 degrees
- moved R5 16.5 mm to (40.6, 40.0), turned to 270 degrees
- moved R8 16.5 mm to (14.0, 40.0), turned to 270 degrees
- moved R10 16.1 mm to (10.2, 40.0), turned to 270 degrees
- moved R12 16.1 mm to (21.6, 40.0), turned to 270 degrees
- moved R13 16.1 mm to (25.4, 40.0), turned to 270 degrees
- moved R3 16.1 mm to (44.5, 40.0), turned to 270 degrees
- moved R9 16.1 mm to (6.35, 40.0), turned to 270 degrees
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- renumbered U$2 to U9, U$3 to U10
Connections:
- removed net DISP_SEL2: R20.1
- removed net LED: LED1.A
- removed net MOSI0: U1.15, U9.5
- removed net N$32: POT4.P$2, U3.W1
- removed net N$33: POT5.P$1, U3.B2
- removed net N$34: POT5.P$3, U3.A2
- removed net N$35: POT5.P$2, U3.W2
- new net MOSI0/LED: LED1.A, U1.15, U9.5
- new net N$14: POT2.P$2, U3.W2
- new net N$15: POT1.P$2, U2.W1
- new net N$16: POT0.P$2, U2.W2
- new net N$17: POT4.P$2, U4.W2
- net DISP_2: now also U6.E1, U6.E2; no longer U6.C1, U6.C2
- net DISP_4: now also U6.C1, U6.C2; no longer U6.E1, U6.E2
- net DISP_SEL1: now also R20.1
- net N$18: now also POT5.P$2; no longer POT0.P$2
- net N$19: now also POT3.P$2, U3.W1; no longer POT0.P$1, U4.B1
- net N$20: now also U2.A2; no longer U4.A1
- net N$21: now also POT0.P$1, U2.B2; no longer POT1.P$1, U4.B2
- net N$22: now also POT3.P$1, U3.B1; no longer POT1.P$3, U4.A2
- net N$23: now also POT3.P$3, U3.A1; no longer POT1.P$2, U4.W2
- net N$24: now also U3.B2; no longer U2.B1
- net N$25: now also U3.A2; no longer U2.A1
- net N$26: now also POT1.P$1, U2.B1; no longer POT2.P$2, U2.W1
- net N$27: now also POT1.P$3, U2.A1; no longer POT3.P$1, U2.B2
- net N$28: now also POT4.P$3, U4.A2; no longer POT3.P$3, U2.A2
- net N$29: now also POT5.P$3, U4.A1; no longer POT3.P$2, U2.W2
- net N$30: now also U4.B2; no longer U3.B1
- net N$31: now also POT5.P$1, U4.B1; no longer POT4.P$3, U3.A1
- net S1: now also SW1.P$2; no longer SW0.P$2
- net S1A: now also SW1.P$1; no longer SW0.P$1
- net S1B: now also SW1.P$3; no longer SW0.P$3
- net S2: now also SW0.P$2; no longer SW1.P$2
- net S2A: now also SW0.P$1; no longer SW1.P$1
- net S2B: now also SW0.P$3; no longer SW1.P$3
Routing:
- net VDD: track 0.00 -> 297.0 mm, vias 0 -> 8
- net GND: track 0.00 -> 96.3 mm, vias 0 -> 13
- net INPUT_2: track 0.00 -> 81.0 mm
- net I2C1_SCL: track 0.00 -> 75.3 mm, vias 0 -> 4
- net ENC_SW: track 0.00 -> 74.9 mm, vias 0 -> 2
- net INPUT_5: track 0.00 -> 74.1 mm
- net INPUT_1: track 0.00 -> 71.8 mm
- net RESET: track 0.00 -> 71.5 mm, vias 0 -> 2
- net I2C1_SDA: track 0.00 -> 67.5 mm, vias 0 -> 4
- net INPUT_4: track 0.00 -> 63.9 mm
- net INPUT_0: track 0.00 -> 62.9 mm
- net DISP_6: track 0.00 -> 58.0 mm, vias 0 -> 1
- net DISP_7: track 0.00 -> 54.5 mm
- net DISP_5: track 0.00 -> 54.1 mm, vias 0 -> 1
- net INPUT_3: track 0.00 -> 53.6 mm
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- added copper zone on layer 15, net GND
Other:
- board size 61 x 64.1 mm -> 61 x 64 mm
- board text added: "PARASITE"
- board text added: "U8"
